Commit message: Add files via upload

File: hexapod_description/urdf/hexapod1.urdf (robot description, URDF)
Before this commit: robot hexapod, 19 links, 18 joints
Links:
- link base_link: geometry collision cylinder length=0.05 radius=0.22; visual cylinder length=0.05 radius=0.22
Joints:
- joint leg1_hip_yaw: origin xyz=0.15 0.15 -0.025 rpy=0 0 0 -> xyz=0.22 0.0 -0.025 rpy=0 0 0.0
- joint leg2_hip_yaw: origin xyz=0.15 -0.15 -0.025 rpy=0 0 0 -> xyz=0.11 0.190525588 -0.025 rpy=0 0 1.0472
- joint leg3_hip_yaw: origin xyz=0.0 0.18 -0.025 rpy=0 0 0 -> xyz=-0.11 0.190525588 -0.025 rpy=0 0 2.0944
- joint leg4_hip_yaw: origin xyz=0.0 -0.18 -0.025 rpy=0 0 0 -> xyz=-0.22 0.0 -0.025 rpy=0 0 3.1416
- joint leg5_hip_yaw: origin xyz=-0.15 0.15 -0.025 rpy=0 0 0 -> xyz=-0.11 -0.190525588 -0.025 rpy=0 0 -2.0944
- joint leg6_hip_yaw: origin xyz=-0.15 -0.15 -0.025 rpy=0 0 0 -> xyz=0.11 -0.190525588 -0.025 rpy=0 0 -1.0472
